Commit message: URDF representation of the Quanser QArm
Added the rotation limits for the 4 revolute joints.

File: urdf/QARM.urdf (robot description, URDF)
Before this commit: robot QARM, 6 links, 5 joints
Joints:
- joint ELBOW: axis 0 0 -1 -> 0 0 1; limit lower=0 upper=0 effort=0 velocity=0 -> lower=-1.658 upper=1.309 effort=0 velocity=0
- joint SHOULDER: limit lower=0 upper=0 effort=0 velocity=0 -> lower=-1.483 upper=1.483 effort=0 velocity=0
- joint WRIST: limit lower=0 upper=0 effort=0 velocity=0 -> lower=-3.010 upper=3.010 effort=0 velocity=0
- joint YAW: limit lower=0 upper=0 effort=0 velocity=0 -> lower=-2.967 upper=2.967 effort=0 velocity=0
